File: protea/esp8266.kicad_sch (KiCad schematic)
At the start: 10 parts, among them J5 ESP8266 Prog, U5 ESP8266-12E_ESP-12E

Commit message: Protea 1.1 WIP
Parts:
- S3: renamed from S4; footprint FRANK:Button (SMD, 3x3mm, 1-1) -> FRANK:TACT-SIDE-4623
- S4: renamed from S5; footprint FRANK:Button (SMD, 3x3mm, 1-1) -> FRANK:TACT-SIDE-4623
- renumbered J5 to J4, R20 to R17, R21 to R18, R22 to R19, R24 to R20, R23 to R21, U5 to U8
Changed lines of the file:
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@@
 	(title_block
 		(title "${NAME}")
-		(date "2025-04-21")
+		(date "2025-05-25")
 		(rev "${VERSION}")
 		(company "Mikhail Matveev")
@@
 			(width 0)
 			(type default)
+		)
+	)
+	(label "TXD"
+		(at 167.64 62.23 180)
+		(effects
+			(font
+				(size 1.27 1.27)
+			)
+			(justify right bottom)
+		)
+	)
+	(label "RXD"
+		(at 123.19 109.22 180)
+		(effects
+			(font
+				(size 1.27 1.27)
+			)
+			(justify right bottom)
+		)
+	)
+	(label "TXD"
+		(at 123.19 111.76 180)
+		(effects
+			(font
+				(size 1.27 1.27)
+			)
+			(justify right bottom)
 		)
 	)
@@
 		)
 	)
-	(hierarchical_label "RXD"
-		(shape input)
-		(at 123.19 109.22 0)
-		(effects
-			(font
-				(size 1.27 1.27)
-			)
-			(justify left)
-		)
-	)
 	(hierarchical_label "GPIO4"
 		(shape input)
@@
 			)
 			(justify right)
-		)
-	)
-	(hierarchical_label "TXD"
-		(shape input)
-		(at 123.19 111.76 0)
-		(effects
-			(font
-				(size 1.27 1.27)
-			)
-			(justify left)
 		)
 	)
@@
 		(dnp no)
 		(fields_autoplaced yes)
-		(property "Reference" "#PWR047"
+		(property "Reference" "#PWR055"
 			(at 82.55 62.23 0)
 			(effects
@@
 			(project "protea"
 				(path "/8c0b3d8b-46d3-4173-ab1e-a61765f77d61/a87f9c19-f253-403f-87e9-05ed3e46708d"
-					(reference "#PWR047")
+					(reference "#PWR055")
 					(unit 1)
 				)
@@
 		(on_board yes)
 		(dnp no)
-		(property "Reference" "R20"
+		(property "Reference" "R17"
 			(at 65.8622 50.8 90)
 			(effects
@@
 			(project "protea"
 				(path "/8c0b3d8b-46d3-4173-ab1e-a61765f77d61/a87f9c19-f253-403f-87e9-05ed3e46708d"
-					(reference "R20")
+					(reference "R17")
 					(unit 1)
 				)
@@
 		(dnp no)
 		(fields_autoplaced yes)
-		(property "Reference" "J5"
+		(property "Reference" "J4"
 			(at 108.585 104.14 0)
 			(effects
@@
 			(project ""
 				(path "/8c0b3d8b-46d3-4173-ab1e-a61765f77d61/a87f9c19-f253-403f-87e9-05ed3e46708d"
-					(reference "J5")
+					(reference "J4")
 					(unit 1)
 				)
@@
 		(on_board yes)
 		(dnp no)
-		(property "Reference" "R21"
+		(property "Reference" "R18"
 			(at 87.8078 62.23 90)
 			(effects
@@
 			(project "protea"
 				(path "/8c0b3d8b-46d3-4173-ab1e-a61765f77d61/a87f9c19-f253-403f-87e9-05ed3e46708d"
-					(reference "R21")
+					(reference "R18")
 					(unit 1)
 				)
@@
 		(dnp no)
 		(fields_autoplaced yes)
-		(property "Reference" "#PWR055"
+		(property "Reference" "#PWR060"
 			(at 201.93 87.63 0)
 			(effects
@@
 			(project "protea"
 				(path "/8c0b3d8b-46d3-4173-ab1e-a61765f77d61/a87f9c19-f253-403f-87e9-05ed3e46708d"
-					(reference "#PWR055")
+					(reference "#PWR060")
 					(unit 1)
 				)
@@
 		(dnp no)
 		(fields_autoplaced yes)
-		(property "Reference" "#PWR050"
+		(property "Reference" "#PWR058"
 			(at 71.12 82.55 0)
 			(effects
@@
 			(project "protea"
 				(path "/8c0b3d8b-46d3-4173-ab1e-a61765f77d61/a87f9c19-f253-403f-87e9-05ed3e46708d"
-					(reference "#PWR050")
+					(reference "#PWR058")
 					(unit 1)
 				)
@@
 		(on_board yes)
 		(dnp no)
-		(property "Reference" "R24"
+		(property "Reference" "R20"
 			(at 76.3778 82.55 90)
 			(effects
@@
 			(project "protea"
 				(path "/8c0b3d8b-46d3-4173-ab1e-a61765f77d61/a87f9c19-f253-403f-87e9-05ed3e46708d"
-					(reference "R24")
+					(reference "R20")
 					(unit 1)
 				)
@@
 		(dnp no)
 		(fields_autoplaced yes)
-		(property "Reference" "#PWR046"
+		(property "Reference" "#PWR054"
 			(at 71.12 72.39 0)
 			(effects
@@
 			(project "protea"
 				(path "/8c0b3d8b-46d3-4173-ab1e-a61765f77d61/a87f9c19-f253-403f-87e9-05ed3e46708d"
-					(reference "#PWR046")
+					(reference "#PWR054")
 					(unit 1)
 				)
@@
 		(dnp no)
 		(fields_autoplaced yes)
-		(property "Reference" "#PWR044"
+		(property "Reference" "#PWR051"
 			(at 162.56 35.56 0)
 			(effects
@@
 			(project ""
 				(path "/8c0b3d8b-46d3-4173-ab1e-a61765f77d61/a87f9c19-f253-403f-87e9-05ed3e46708d"
-					(reference "#PWR044")
+					(reference "#PWR051")
 					(unit 1)
 				)
@@
 		(dnp no)
 		(fields_autoplaced yes)
-		(property "Reference" "#PWR048"
+		(property "Reference" "#PWR057"
 			(at 201.93 80.01 0)
 			(effects
@@
 			(project "protea"
 				(path "/8c0b3d8b-46d3-4173-ab1e-a61765f77d61/a87f9c19-f253-403f-87e9-05ed3e46708d"
-					(reference "#PWR048")
+					(reference "#PWR057")
 					(unit 1)
 				)
@@
 		(dnp no)
 		(fields_autoplaced yes)
-		(property "Reference" "S4"
+		(property "Reference" "S3"
 			(at 72.39 58.4199 90)
 			(effects
@@
 			)
 		)
-		(property "Footprint" "FRANK:Button (SMD, 3x3mm, 1-1)"
+		(property "Footprint" "FRANK:TACT-SIDE-4623"
 			(at 66.04 59.69 0)
 			(effects
@@
 			(project "protea"
 				(path "/8c0b3d8b-46d3-4173-ab1e-a61765f77d61/a87f9c19-f253-403f-87e9-05ed3e46708d"
-					(reference "S4")
+					(reference "S3")
 					(unit 1)
 				)
@@
 		(dnp no)
 		(fields_autoplaced yes)
-		(property "Reference" "S5"
+		(property "Reference" "S4"
 			(at 57.15 67.31 0)
 			(effects
@@
 			)
 		)
-		(property "Footprint" "FRANK:Button (SMD, 3x3mm, 1-1)"
+		(property "Footprint" "FRANK:TACT-SIDE-4623"
 			(at 57.15 69.85 0)
 			(effects
@@
 			(project "protea"
 				(path "/8c0b3d8b-46d3-4173-ab1e-a61765f77d61/a87f9c19-f253-403f-87e9-05ed3e46708d"
-					(reference "S5")
+					(reference "S4")
 					(unit 1)
 				)
@@
 		(dnp no)
 		(fields_autoplaced yes)
-		(property "Reference" "#PWR049"
+		(property "Reference" "#PWR059"
 			(at 90.17 82.55 0)
 			(effects
@@
 			(project "protea"
 				(path "/8c0b3d8b-46d3-4173-ab1e-a61765f77d61/a87f9c19-f253-403f-87e9-05ed3e46708d"
-					(reference "#PWR049")
+					(reference "#PWR059")
 					(unit 1)
 				)
@@
 		(on_board yes)
 		(dnp no)
-		(property "Reference" "R23"
+		(property "Reference" "R21"
 			(at 95.4278 82.55 90)
 			(effects
@@
 			(project "protea"
 				(path "/8c0b3d8b-46d3-4173-ab1e-a61765f77d61/a87f9c19-f253-403f-87e9-05ed3e46708d"
-					(reference "R23")
+					(reference "R21")
 					(unit 1)
 				)
@@
 		(dnp no)
 		(fields_autoplaced yes)
-		(property "Reference" "#PWR051"
+		(property "Reference" "#PWR056"
 			(at 44.45 74.93 0)
 			(effects
@@
 			(project "protea"
 				(path "/8c0b3d8b-46d3-4173-ab1e-a61765f77d61/a87f9c19-f253-403f-87e9-05ed3e46708d"
-					(reference "#PWR051")
+					(reference "#PWR056")
 					(unit 1)
 				)
@@
 		(dnp no)
 		(fields_autoplaced yes)
-		(property "Reference" "#PWR043"
+		(property "Reference" "#PWR053"
 			(at 166.37 54.61 0)
 			(effects
@@
 			(project ""
 				(path "/8c0b3d8b-46d3-4173-ab1e-a61765f77d61/a87f9c19-f253-403f-87e9-05ed3e46708d"
-					(reference "#PWR043")
+					(reference "#PWR053")
 					(unit 1)
 				)
@@
 		(on_board yes)
 		(dnp no)
-		(property "Reference" "R22"
+		(property "Reference" "R19"
 			(at 187.96 74.7522 90)
 			(effects
@@
 			(project "protea"
 				(path "/8c0b3d8b-46d3-4173-ab1e-a61765f77d61/a87f9c19-f253-403f-87e9-05ed3e46708d"
-					(reference "R22")
+					(reference "R19")
 					(unit 1)
 				)
@@
 		(dnp no)
 		(fields_autoplaced yes)
-		(property "Reference" "U5"
+		(property "Reference" "U8"
 			(at 139.7 46.99 0)
 			(effects
@@
 			(project ""
 				(path "/8c0b3d8b-46d3-4173-ab1e-a61765f77d61/a87f9c19-f253-403f-87e9-05ed3e46708d"
-					(reference "U5")
+					(reference "U8")
 					(unit 1)
 				)
@@
 		(dnp no)
 		(fields_autoplaced yes)
-		(property "Reference" "#PWR045"
+		(property "Reference" "#PWR052"
 			(at 71.12 50.8 0)
 			(effects
@@
 			(project "protea"
 				(path "/8c0b3d8b-46d3-4173-ab1e-a61765f77d61/a87f9c19-f253-403f-87e9-05ed3e46708d"
-					(reference "#PWR045")
+					(reference "#PWR052")
 					(unit 1)
 				)
@@
 		(on_board yes)
 		(dnp no)
-		(property "Reference" "#PWR052"
+		(property "Reference" "#PWR061"
 			(at 128.27 114.3 0)
 			(effects
@@
 			(project "protea"
 				(path "/8c0b3d8b-46d3-4173-ab1e-a61765f77d61/a87f9c19-f253-403f-87e9-05ed3e46708d"
-					(reference "#PWR052")
+					(reference "#PWR061")
 					(unit 1)
 				)
