File: protea/esp8266.kicad_sch (KiCad schematic)
At the start: 10 parts, among them J4 ESP8266 Prog, U8 ESP8266-12E_ESP-12E

Commit message: Protea HW 2.06
Parts:
- J4: AliExpress (none) -> https://vi.aliexpress.com/item/1005006186853439.html
- U8: value ESP8266-12E_ESP-12E -> ESP8266 ESP-12F; AliExpress (none) -> https://vi.aliexpress.com/item/1005007014587323.html
Other:
- moved on the sheet: C24, J4, R17, R18, R19, R20, R21, S3, S4, U8
