File: protea/hdmi.kicad_sch (KiCad schematic)
At the start: 10 parts, among them J4 HDMI Female

Commit message: Protea 1.1 WIP
Parts:
- renumbered C23 to C25, J4 to J5, R12 to R22, R13 to R23, R14 to R24, R15 to R25, R16 to R26, R17 to R27, R18 to R28, R19 to R29
Changed lines of the file:
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@@
 	(title_block
 		(title "${NAME}")
-		(date "2025-04-21")
+		(date "2025-05-25")
 		(rev "${VERSION}")
 		(company "Mikhail Matveev")
@@
 		(on_board yes)
 		(dnp no)
-		(property "Reference" "R15"
+		(property "Reference" "R25"
 			(at 90.17 104.14 90)
 			(effects
@@
 			(project "frank2"
 				(path "/8c0b3d8b-46d3-4173-ab1e-a61765f77d61/1ea0e9ac-8f42-4d3d-8b47-067d751f5a51"
-					(reference "R15")
+					(reference "R25")
 					(unit 1)
 				)
@@
 		(on_board yes)
 		(dnp no)
-		(property "Reference" "R17"
+		(property "Reference" "R27"
 			(at 100.33 111.76 90)
 			(effects
@@
 			(project "frank2"
 				(path "/8c0b3d8b-46d3-4173-ab1e-a61765f77d61/1ea0e9ac-8f42-4d3d-8b47-067d751f5a51"
-					(reference "R17")
+					(reference "R27")
 					(unit 1)
 				)
@@
 		(on_board yes)
 		(dnp no)
-		(property "Reference" "R12"
+		(property "Reference" "R22"
 			(at 90.17 91.44 90)
 			(effects
@@
 			(project "frank2"
 				(path "/8c0b3d8b-46d3-4173-ab1e-a61765f77d61/1ea0e9ac-8f42-4d3d-8b47-067d751f5a51"
-					(reference "R12")
+					(reference "R22")
 					(unit 1)
 				)
@@
 		(dnp no)
 		(fields_autoplaced yes)
-		(property "Reference" "#PWR040"
+		(property "Reference" "#PWR062"
 			(at 71.12 81.28 0)
 			(effects
@@
 			(project ""
 				(path "/8c0b3d8b-46d3-4173-ab1e-a61765f77d61/1ea0e9ac-8f42-4d3d-8b47-067d751f5a51"
-					(reference "#PWR040")
+					(reference "#PWR062")
 					(unit 1)
 				)
@@
 		(on_board yes)
 		(dnp no)
-		(property "Reference" "R16"
+		(property "Reference" "R26"
 			(at 90.17 106.68 90)
 			(effects
@@
 			(project "frank2"
 				(path "/8c0b3d8b-46d3-4173-ab1e-a61765f77d61/1ea0e9ac-8f42-4d3d-8b47-067d751f5a51"
-					(reference "R16")
+					(reference "R26")
 					(unit 1)
 				)
@@
 		(on_board yes)
 		(dnp no)
-		(property "Reference" "C23"
+		(property "Reference" "C25"
 			(at 76.3016 74.549 0)
 			(effects
@@
 			(project "frank2"
 				(path "/8c0b3d8b-46d3-4173-ab1e-a61765f77d61/1ea0e9ac-8f42-4d3d-8b47-067d751f5a51"
-					(reference "C23")
+					(reference "C25")
 					(unit 1)
 				)
@@
 		(on_board yes)
 		(dnp no)
-		(property "Reference" "R14"
+		(property "Reference" "R24"
 			(at 80.01 99.06 90)
 			(effects
@@
 			(project "frank2"
 				(path "/8c0b3d8b-46d3-4173-ab1e-a61765f77d61/1ea0e9ac-8f42-4d3d-8b47-067d751f5a51"
-					(reference "R14")
+					(reference "R24")
 					(unit 1)
 				)
@@
 		(dnp no)
 		(fields_autoplaced yes)
-		(property "Reference" "#PWR042"
+		(property "Reference" "#PWR064"
 			(at 67.31 137.16 0)
 			(effects
@@
 			(project "frank2"
 				(path "/8c0b3d8b-46d3-4173-ab1e-a61765f77d61/1ea0e9ac-8f42-4d3d-8b47-067d751f5a51"
-					(reference "#PWR042")
+					(reference "#PWR064")
 					(unit 1)
 				)
@@
 		(dnp no)
 		(fields_autoplaced yes)
-		(property "Reference" "#PWR041"
+		(property "Reference" "#PWR063"
 			(at 87.63 77.47 0)
 			(effects
@@
 			(project ""
 				(path "/8c0b3d8b-46d3-4173-ab1e-a61765f77d61/1ea0e9ac-8f42-4d3d-8b47-067d751f5a51"
-					(reference "#PWR041")
+					(reference "#PWR063")
 					(unit 1)
 				)
@@
 		(on_board yes)
 		(dnp no)
-		(property "Reference" "R13"
+		(property "Reference" "R23"
 			(at 100.33 96.52 90)
 			(effects
@@
 			(project "frank2"
 				(path "/8c0b3d8b-46d3-4173-ab1e-a61765f77d61/1ea0e9ac-8f42-4d3d-8b47-067d751f5a51"
-					(reference "R13")
+					(reference "R23")
 					(unit 1)
 				)
@@
 		(dnp no)
 		(fields_autoplaced yes)
-		(property "Reference" "J4"
+		(property "Reference" "J5"
 			(at 43.18 91.4399 0)
 			(effects
@@
 			(project "frank2"
 				(path "/8c0b3d8b-46d3-4173-ab1e-a61765f77d61/1ea0e9ac-8f42-4d3d-8b47-067d751f5a51"
-					(reference "J4")
+					(reference "J5")
 					(unit 1)
 				)
@@
 		(on_board yes)
 		(dnp no)
-		(property "Reference" "R19"
+		(property "Reference" "R29"
 			(at 90.17 119.38 90)
 			(effects
@@
 			(project "frank2"
 				(path "/8c0b3d8b-46d3-4173-ab1e-a61765f77d61/1ea0e9ac-8f42-4d3d-8b47-067d751f5a51"
-					(reference "R19")
+					(reference "R29")
 					(unit 1)
 				)
@@
 		(on_board yes)
 		(dnp no)
-		(property "Reference" "R18"
+		(property "Reference" "R28"
 			(at 80.01 114.3 90)
 			(effects
@@
 			(project "frank2"
 				(path "/8c0b3d8b-46d3-4173-ab1e-a61765f77d61/1ea0e9ac-8f42-4d3d-8b47-067d751f5a51"
-					(reference "R18")
+					(reference "R28")
 					(unit 1)
 				)
