File: protea/power.kicad_sch (KiCad schematic)
At the start: 9 parts, among them J1 USB4215-03-A, U1 NCP1117 3.3

Commit message: Protea 1.1 WIP
Parts:
- added R3, R4: 22R, FRANK:Resistor (0805), symbol Device:R
- added U3: USBLC6-2SC6, FRANK:SOT-23-6, symbol FRANK:USBLC6-2SC6
- J1: LCSC C165948 -> (none)
- LD1: value Green -> Power
- R2: renamed from R1; LCSC (none) -> (none)
- R5: renamed from R3; LCSC (none) -> (none)
- renumbered C1 to C3, R4 to R6, R2 to R7, U1 to U2
Connections:
- net D+: now also U3.4 (I/O2); no longer J1.6 (DP1), J1.8 (DP2)
- net D-: now also U3.6 (I/O1); no longer J1.5 (DN2), J1.7 (DN1)
- net GND: now also U3.2 (GND)
- net VBUS: now also U3.5 (VBUS)
- new net: R3.1, U3.1 (I/O1)
- new net: R4.1, U3.3 (I/O2)
- new net: J1.5 (DN2), J1.7 (DN1), R3.2
- new net: J1.6 (DP1), J1.8 (DP2), R4.2
Other:
- title: ${NAME} -> MiniFRANK RM1P2
- moved on the sheet: C2, C3, LD1, R2, R5, R6, R7, U2
