File: protea/power.kicad_sch (KiCad schematic)
At the start: 12 parts, among them J1 USB4215-03-A, U2 NCP1117 3.3, U3 USBLC6-2SC6

Commit message: Protea HW 2.06
Parts:
- LD1: value Power -> Green
- R7: AliExpress https://www.vishay.com/docs/28952/mcs0402at-mct0603at-mcu08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 -> https://www.aliexpress.com/item/1005005945735199.html
- U3: AliExpress (none) -> https://vi.aliexpress.com/item/1005006883533480.html
Other:
- title: MiniFRANK RM1P2 -> ${NAME}
Changed lines of the file:
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@@
 	(paper "A4")
 	(title_block
-		(title "MiniFRANK RM1P2")
-		(date "2025-05-24")
+		(title "${NAME}")
+		(date "2025-05-26")
 		(rev "${VERSION}")
 		(company "Mikhail Matveev")
@@
 			)
 		)
+		(property "AliExpress" "https://vi.aliexpress.com/item/1005006883533480.html"
+			(at 148.59 90.17 0)
+			(effects
+				(font
+					(size 1.27 1.27)
+				)
+				(hide yes)
+			)
+		)
 		(pin "2"
 		)
@@
 			)
 		)
-		(property "Value" "Power"
+		(property "Value" "Green"
 			(at 183.8325 115.57 0)
 			(effects
@@
 			)
 		)
-		(property "AliExpress" "https://www.vishay.com/docs/28952/mcs0402at-mct0603at-mcu0805at-mca1206at.pdf"
+		(property "AliExpress" "https://www.aliexpress.com/item/1005005945735199.html"
 			(at 193.04 119.38 0)
 			(effects
