File: protea/protea.kicad_pcb (KiCad board)
At the start: 2 copper layers, 84 x 47.5 mm, 91 parts, among them J1 USB4215-03-A, J2 D-SUB 9 Male, J3 676430910, J4 ESP8266 Prog, J5 HDMI Female, U1 SN74CBT3257CDR, U10 TS3USB221RSER, U2 NCP1117 3.3, U3 USBLC6-2SC6, U4 W25Q128JVSIQ, U5 RP2040, U6 MAX232CSE+, U7 USBLC6-2SC6, U8 ESP8266-12E_ESP-12E, U9 CH340C, Y1 12 MHz

Commit message: Protea 1.01 WIP
Parts:
- moved C23 2.43 mm to (197.8, 59.2), turned to -90 degrees
- moved C25 1.52 mm to (195.2, 59.2)
Routing:
- net /ESP_TXD: track 0.00 -> 82.2 mm, vias 0 -> 3
- net /ESP_RXD: track 0.00 -> 69.5 mm, vias 0 -> 3
- net /UT_D-: track 0.00 -> 49.1 mm, vias 0 -> 2
- net /UT_D+: track 0.00 -> 46.6 mm, vias 0 -> 2
- net /SN74_S: track 0.00 -> 44.5 mm, vias 0 -> 4
- net Net-(U8-RESET): track 0.00 -> 44.3 mm, vias 0 -> 2
- net Net-(U8-IO0): track 0.00 -> 35.5 mm, vias 0 -> 2
- net /GPIO14: track 2.38 -> 35.5 mm, vias 1 -> 2
- net /RS232/RTS_IN: track 0.00 -> 29.8 mm, vias 0 -> 1
- net /RS232/CTS_MAX: track 0.00 -> 27.1 mm, vias 0 -> 2
- net /RS232_TX: track 0.00 -> 26.3 mm, vias 0 -> 2
- net Net-(R9-Pad2): track 0.00 -> 23.6 mm, vias 0 -> 2
- net /RS232_RTS: track 0.00 -> 22.8 mm, vias 0 -> 2
- net /RS232/CTS_IN: track 0.00 -> 21.5 mm, vias 0 -> 1
- net /RS232/TX_IN: track 0.00 -> 21.2 mm, vias 0 -> 1
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Other:
- outline, holes or cut-outs redrawn
- board text added: "D"
- board text added: "ESP BOOT"
- board text added: "ESP RESET"
- board text added: "GND"
- board text added: "M"
- board text added: "RP BOOT"
- board text added: "RP RESET"
- board text added: "RX"
- board text added: "TX"
- board text added: "U"

Commit message: Protea WIP
Parts:
- U6: footprint FRANK:SOIC127P600X175-16N -> FRANK:SOP-16
Routing:
- net /PW_D-: track 9.94 -> 12.5 mm
- net /RS232_TX: track 26.3 -> 28.6 mm
- net Net-(J2-Pad1): track 12.2 -> 13.3 mm
- net /RS232/V+: track 4.59 -> 5.63 mm

Commit message: Protea HW 2.06
Parts:
- JP1: value Main Jumpers -> DS05-127-2-03BK-SMT-TR
- LD1: value Power -> Green
- LD2: value BLUE -> Blue
- LD3: value TX -> Orange
- LD4: value RX -> Orange
- U8: value ESP8266-12E_ESP-12E -> ESP8266 ESP-12F
- Y1: value 12 MHz -> 12 MHz Passive
- moved LD1 78.7 mm to (147.8, 57.0)
- moved R7 78.6 mm to (147.8, 59.8)
Routing:
- net /PW_D+: track 10.6 -> 5.87 mm, vias 0 -> 2
- net /UT_D-: track 49.1 -> 46.0 mm
- net Net-(U9-3V): track 20.4 -> 22.5 mm
- net +3V3: track 212.9 -> 215.0 mm, vias 9 -> 8
- net /UT_D+: track 46.6 -> 48.4 mm
- net /RS232/TX_IN: track 21.6 -> 19.9 mm
- net VBUS: track 174.7 -> 175.9 mm
- net /RP2040/QSPI_SD3: track 28.9 -> 27.7 mm
- net /RS232_VBUS: track 4.13 -> 3.11 mm
- net /RS232/RX_IN: track 21.0 -> 20.0 mm
- net /GPIO14: track 35.5 -> 36.5 mm
- net Net-(J5-D2P): track 6.39 -> 7.26 mm
- net /RP_D+: track 38.1 -> 38.7 mm
- net GND: vias 38 -> 37
Other:
- board text added: "${NAME}"
- board text added: "${VERSION}"
- board text added: "rh1.tech"
