File: protea/protea.kicad_sch (KiCad schematic)
At the start: 6 parts, among them J6 SD04H0SB

Commit message: Protea 1.1 WIP
Parts:
- removed J6: SD04H0SB, FRANK:DIP Switch (5x5), symbol Connector_Generic:Conn_02x05_Odd_Even
- removed S1: Reset, FRANK:Button (SMD, 3x3mm, 1-1), symbol Switch:SW_Push
- added C1: 100n, FRANK:Capacitor (0805), symbol Device:C
- added JP1: Main Jumpers, FRANK:DS05127203BKSMTTR, symbol Switch:SW_DIP_x03
- added R1: 10K, FRANK:Resistor (0805), symbol Device:R
- added U1: SN74CBT3257CDR, FRANK:SOP-16, symbol FRANK:SN74CBT3257CDR
Connections:
- net ESP_RXD: now also U1.2 (1B1)
- net ESP_TXD: now also U1.5 (2B1)
- net GND: now also C1.1, JP1.4, JP1.5, R1.1, U1.11 (3B1), U1.14 (4B1), U1.15 (~{OE}), U1.8 (GND)
- net GPIO14: now also JP1.2
- net GPIO16: now also U1.4 (1A)
- net GPIO17: now also U1.7 (2A)
- net GPIO18: now also U1.9 (3A)
- net GPIO19: now also U1.12 (4A)
- net VBUS: now also C1.2, JP1.6, U1.16 (VCC)
- new net RS232_CTS: U1.10 (3B2)
- new net RS232_RTS: U1.13 (4B2)
- new net RS232_RX: U1.6 (2B2)
- new net RS232_TX: U1.3 (1B2)
- new net SN74_S: JP1.1, R1.2, U1.1 (S)
- new net USBMPXSW: JP1.3
- no-connect marks 38 -> 37
Other:
- added sheet USB Multiplexer (usb_multiplexer.kicad_sch)
- added sheet USB to TTL (usb2ttl.kicad_sch)
- note added: "GPIO18"
- note added: "GPIO19"
- note removed: "Defaults"
- note removed: "HDMI Jumper"
