File: protea/protea.kicad_sch (KiCad schematic)
At the start: 8 parts, among them U1 SN74CBT3257CDR

Commit message: Protea HW 2.06
Parts:
- JP1: value Main Jumpers -> DS05-127-2-03BK-SMT-TR
- U1: AliExpress (none) -> https://vi.aliexpress.com/item/1005008608415566.html
Other:
- note removed: "GPIO16"
- note removed: "GPIO17"
- note removed: "GPIO18"
- note removed: "GPIO19"
- moved on the sheet: C1, JP1, R1, U1
