File: protea/rp2040.kicad_sch (KiCad schematic)
At the start: 25 parts, among them U2 W25Q128JVSIQ, U3 RP2040, Y1 12 MHz

Commit message: Protea 1.1 WIP
Parts:
- added S2: Reset, FRANK:TACT-SIDE-4623, symbol Switch:SW_Push
- S1: renamed from S3; footprint FRANK:Button (SMD, 3x3mm, 1-1) -> FRANK:TACT-SIDE-4623
- renumbered C9 to C10, C10 to C11, C11 to C12, C12 to C13, C13 to C14, C14 to C15, C15 to C16, C16 to C17, C17 to C18, C3 to C4, C4 to C5, C5 to C6, C6 to C7, C7 to C8, C8 to C9, R7 to R10, R8 to R11, R9 to R12, R5 to R8, R6 to R9, U2 to U4, U3 to U5
Connections:
- net GND: now also S2.2
- net RUN: now also S2.1
