File: protea/rs232.kicad_sch (KiCad schematic)
At the start: 10 parts, among them J2 D-SUB 9 Male, U4 MAX232CSE+

Commit message: Protea 1.1 WIP
Parts:
- renumbered C18 to C19, C19 to C20, C20 to C21, C21 to C22, R10 to R13, R11 to R14, U4 to U6
Changed lines of the file:
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@@
 	(title_block
 		(title "${NAME}")
-		(date "2025-04-21")
+		(date "2025-05-25")
 		(rev "${VERSION}")
 		(company "Mikhail Matveev")
@@
 		(dnp no)
 		(fields_autoplaced yes)
-		(property "Reference" "C19"
+		(property "Reference" "C20"
 			(at 59.6963 62.23 90)
 			(effects
@@
 			(project "turbofrank"
 				(path "/8c0b3d8b-46d3-4173-ab1e-a61765f77d61/743e81f1-e5ae-4430-9dee-0c06cb416437"
-					(reference "C19")
+					(reference "C20")
 					(unit 1)
 				)
@@
 		(dnp no)
 		(fields_autoplaced yes)
-		(property "Reference" "#PWR031"
+		(property "Reference" "#PWR041"
 			(at 99.06 36.83 0)
 			(effects
@@
 			(project ""
 				(path "/8c0b3d8b-46d3-4173-ab1e-a61765f77d61/743e81f1-e5ae-4430-9dee-0c06cb416437"
-					(reference "#PWR031")
+					(reference "#PWR041")
 					(unit 1)
 				)
@@
 		(dnp no)
 		(fields_autoplaced yes)
-		(property "Reference" "C20"
+		(property "Reference" "C21"
 			(at 48.2663 67.31 90)
 			(effects
@@
 			(project "turbofrank"
 				(path "/8c0b3d8b-46d3-4173-ab1e-a61765f77d61/743e81f1-e5ae-4430-9dee-0c06cb416437"
-					(reference "C20")
+					(reference "C21")
 					(unit 1)
 				)
@@
 		(dnp no)
 		(fields_autoplaced yes)
-		(property "Reference" "C18"
+		(property "Reference" "C19"
 			(at 106.6863 50.8 90)
 			(effects
@@
 			(project ""
 				(path "/8c0b3d8b-46d3-4173-ab1e-a61765f77d61/743e81f1-e5ae-4430-9dee-0c06cb416437"
-					(reference "C18")
+					(reference "C19")
 					(unit 1)
 				)
@@
 		(dnp no)
 		(fields_autoplaced yes)
-		(property "Reference" "#PWR032"
+		(property "Reference" "#PWR042"
 			(at 146.05 36.83 0)
 			(effects
@@
 			(project "frank2"
 				(path "/8c0b3d8b-46d3-4173-ab1e-a61765f77d61/743e81f1-e5ae-4430-9dee-0c06cb416437"
-					(reference "#PWR032")
+					(reference "#PWR042")
 					(unit 1)
 				)
@@
 		(on_board yes)
 		(dnp no)
-		(property "Reference" "R11"
+		(property "Reference" "R14"
 			(at 144.78 41.91 90)
 			(effects
@@
 			(project "frank2"
 				(path "/8c0b3d8b-46d3-4173-ab1e-a61765f77d61/743e81f1-e5ae-4430-9dee-0c06cb416437"
-					(reference "R11")
+					(reference "R14")
 					(unit 1)
 				)
@@
 		(on_board yes)
 		(dnp no)
-		(property "Reference" "C21"
+		(property "Reference" "C22"
 			(at 46.99 90.17 90)
 			(effects
@@
 			(project "turbofrank"
 				(path "/8c0b3d8b-46d3-4173-ab1e-a61765f77d61/743e81f1-e5ae-4430-9dee-0c06cb416437"
-					(reference "C21")
+					(reference "C22")
 					(unit 1)
 				)
@@
 		(dnp no)
 		(fields_autoplaced yes)
-		(property "Reference" "#PWR033"
+		(property "Reference" "#PWR043"
 			(at 187.96 53.34 0)
 			(effects
@@
 			(project "frank2"
 				(path "/8c0b3d8b-46d3-4173-ab1e-a61765f77d61/743e81f1-e5ae-4430-9dee-0c06cb416437"
-					(reference "#PWR033")
+					(reference "#PWR043")
 					(unit 1)
 				)
@@
 		(dnp no)
 		(fields_autoplaced yes)
-		(property "Reference" "U4"
+		(property "Reference" "U6"
 			(at 96.52 60.96 0)
 			(effects
@@
 			(project "frank2"
 				(path "/8c0b3d8b-46d3-4173-ab1e-a61765f77d61/743e81f1-e5ae-4430-9dee-0c06cb416437"
-					(reference "U4")
+					(reference "U6")
 					(unit 1)
 				)
@@
 		(dnp no)
 		(fields_autoplaced yes)
-		(property "Reference" "#PWR036"
+		(property "Reference" "#PWR045"
 			(at 33.02 83.82 0)
 			(effects
@@
 			(project "frank2"
 				(path "/8c0b3d8b-46d3-4173-ab1e-a61765f77d61/743e81f1-e5ae-4430-9dee-0c06cb416437"
-					(reference "#PWR036")
+					(reference "#PWR045")
 					(unit 1)
 				)
@@
 		(on_board yes)
 		(dnp no)
-		(property "Reference" "R10"
+		(property "Reference" "R13"
 			(at 97.79 41.91 90)
 			(effects
@@
 			(project "frank2"
 				(path "/8c0b3d8b-46d3-4173-ab1e-a61765f77d61/743e81f1-e5ae-4430-9dee-0c06cb416437"
-					(reference "R10")
+					(reference "R13")
 					(unit 1)
 				)
@@
 		(on_board yes)
 		(dnp no)
-		(property "Reference" "#PWR035"
+		(property "Reference" "#PWR044"
 			(at 118.11 71.12 0)
 			(effects
@@
 			(project "frank2"
 				(path "/8c0b3d8b-46d3-4173-ab1e-a61765f77d61/743e81f1-e5ae-4430-9dee-0c06cb416437"
-					(reference "#PWR035")
+					(reference "#PWR044")
 					(unit 1)
 				)
