File: protea/usba.kicad_sch (KiCad schematic)
At the start: 2 parts, among them J3 676430910

Commit message: Protea 1.1 WIP
Parts:
- added R15, R16: 22R, FRANK:Resistor (0805), symbol Device:R
- added U7: USBLC6-2SC6, FRANK:SOT-23-6, symbol FRANK:USBLC6-2SC6
- renumbered C22 to C23
Connections:
- net D+: now also U7.6 (I/O1); no longer J3.3 (D+)
- net D-: now also U7.4 (I/O2); no longer J3.2 (D-)
- net GND: now also U7.2 (GND)
- net VBUS: now also U7.5 (VBUS)
- new net: R15.1, U7.1 (I/O1)
- new net: J3.3 (D+), R15.2
- new net: R16.1, U7.3 (I/O2)
- new net: J3.2 (D-), R16.2
Other:
- moved on the sheet: C23
