File: protea/usb2ttl.kicad_sch (KiCad schematic)
At the start: 7 parts, among them U9 CH340C

Commit message: Protea HW 2.06
Parts:
- C26, C27: AliExpress (none) -> https://www.aliexpress.com/item/33008008276.html
- LD3: value TX -> Orange; AliExpress (none) -> https://www.aliexpress.com/item/1005007252088951.html
- LD4: value RX -> Orange; AliExpress (none) -> https://www.aliexpress.com/item/1005007252088951.html
- R30, R31: AliExpress (none) -> https://www.aliexpress.com/item/1005005945735199.html
- U9: AliExpress (none) -> https://vi.aliexpress.com/item/1005006746838697.html
Other:
- moved on the sheet: C26, C27, LD3, LD4, R30, R31, U9
